Commit message: first commit

File: src/roboticarm_desc/urdf/robotic_arm.urdf (robot description, URDF)
Before this commit: robot roboticarm_desc, 7 links, 6 joints
Links:
- added link tcp_link
Joints:
- added joint tcp_joint: type fixed, parent link_4, child tcp_link, origin xyz=0 0 0.09 rpy=0 0 0

Commit message: pick and place completed with no error

File: src/roboticarm_desc/urdf/robotic_arm.urdf (robot description, URDF)
Before this commit: robot roboticarm_desc, 8 links, 7 joints
Joints:
- joint joint_1: limit lower=0 upper=3.142 effort=300 velocity=3 -> lower=-3.142 upper=3.142 effort=300 velocity=3

Commit message: gazebo added

File: src/roboticarm_desc/urdf/robotic_arm.urdf (robot description, URDF)
Before this commit: robot roboticarm_desc, 8 links, 7 joints
Links:
- link link_1: mass 0.1066908638872 -> 2.066908638872
Joints:
- joint joint_6: mimic joint=joint_5 multiplier=-1 offset=0 -> (none)

File: src/roboticarm_moveit_config/config/roboticarm_desc.ros2_control.xacro (robot description, xacro)
@@ -6,5 +6,6 @@
             <hardware>
                 <!-- By default, set up controllers for simulation. This won't work on real hardware -->
-                <plugin>mock_components/GenericSystem</plugin>
+                <!-- <plugin>mock_components/GenericSystem</plugin> -->
+                  <plugin>gz_ros2_control/GazeboSimSystem</plugin>
                   <param name="mock_sensor_commands">false</param>
                   <param name="state_following_offset">0.0</param>
@@ -45,4 +46,11 @@
                 <state_interface name="velocity"/>
             </joint>
+            <joint name="joint_6">
+                <command_interface name="position"/>
+                <state_interface name="position">
+                <param name="initial_value">${initial_positions['joint_6']}</param>
+                </state_interface>
+                <state_interface name="velocity"/>
+            </joint>
         </ros2_control>
     </xacro:macro>

File: src/roboticarm_moveit_config/config/roboticarm_desc.urdf.xacro (robot description, xacro)
@@ -6,4 +6,19 @@
     <!-- Import control_xacro -->
     <xacro:include filename="roboticarm_desc.ros2_control.xacro" />
-    <xacro:roboticarm_desc_ros2_control name="FakeSystem" initial_positions_file="$(arg initial_positions_file)"/>
+    <gazebo>
+        <plugin filename="gz_ros2_control-system"
+                name="gz_ros2_control::GazeboSimROS2ControlPlugin">
+            <parameters>$(find roboticarm_moveit_config)/config/ros2_controllers.yaml</parameters>
+        </plugin>
+    </gazebo>
+    <gazebo>
+        <plugin filename="gz-sim-joint-mimic-system"
+                name="gz::sim::systems::JointMimic">
+            <joint>joint_5</joint>
+            <mimic_joint>joint_6</mimic_joint>
+            <multiplier>-1</multiplier>
+        </plugin>
+    </gazebo>
+    <!-- <xacro:roboticarm_desc_ros2_control name="FakeSystem" initial_positions_file="$(arg initial_positions_file)"/> -->
+    <xacro:roboticarm_desc_ros2_control name="GazeboSystem" initial_positions_file="$(arg initial_positions_file)"/>
 </robot>
